Commit message: feat: added lidar sensor

File: src/waver_description/urdf/util.xacro (robot description, xacro)
@@ -1,6 +1,11 @@
 <?xml version="1.0"?>
 <robot xmlns:xacro="http://www.ros.org/wiki/xacro" name="waver_utils">
+    <!-- Utils -->
     <xacro:property name="triple_zero" value="0 0 0" />
     <xacro:property name="scale" value="0.001 0.001 0.001" />
+    <xacro:property name="floor_to_top" value="88.5e-03" />
+    <xacro:property name="floor_to_base" value="33.7e-03" />
+    <xacro:property name="base_to_top" value="${ floor_to_top - floor_to_base }" />
+    <xacro:property name="length" value="183e-03" />
     <!-- Base specifications -->
     <xacro:property name="pos_x_base" value="2.838767506182194e-05" />
@@ -76,3 +81,14 @@
     <xacro:property name="mass_center_wbr" value="${pos_x_wbr} ${pos_y_wbr} ${pos_z_wbr}" />
     <xacro:property name="position_wbr" value="${-pos_x_wbr} ${-pos_y_wbr} ${-pos_z_wbr}" />
+    <!-- Lidar specifications -->
+    <xacro:property name="mass_lidar" value="0.05" />
+    <xacro:property name="lidar_model" value="HLS-LFCD-LDS" />
+    <xacro:property name="lidar_link" value="lidar_link" />
+    <xacro:property name="lidar_samples" value="720" />
+    <xacro:property name="lidar_max_range" value="12.0" />
+    <xacro:property name="lidar_min_range" value="0.03" />
+    <xacro:property name="lidar_max_angle" value="${pi}" />
+    <xacro:property name="lidar_min_angle" value="-${pi}" />
+    <xacro:property name="lidar_frequency" value="10" />
+    <xacro:property name="lidar_transform" value="0 0 0 0 0 0" />
 </robot>

File: src/waver_description/urdf/waver.xacro (robot description, xacro)
@@ -5,4 +5,5 @@
   <xacro:include filename="$(find waver_description)/urdf/waver.trans.xacro" />
   <xacro:include filename="$(find waver_description)/urdf/waver.gazebo.xacro" />
+  <xacro:include filename="$(find waver_description)/urdf/lidar.xacro" />
   <!-- ******************************* Links ******************************* -->
   <link name="base_footprint"></link>
@@ -18,5 +19,4 @@
         <mesh filename="package://waver_description/meshes/base_link.stl" scale="${scale}" />
       </geometry>
-      <color rgba="0.1 0.1 0.1 1"/>
       <xacro:dark_gray_material />
     </visual>
