Commit message: refactor: project refactored

File: waver_description/urdf/waver.xacro (robot description, xacro)
@@ -11,9 +11,9 @@
     <inertial>
       <mass value="${mass_base}" />
-      <origin xyz="${mass_center_base}" rpy="0 0 0" />
+      <origin xyz="${mass_center_base}" rpy="0 0 ${pi/2}" />
       <inertia ixx="0.0008255973835920386" iyy="0.0005293282898445326" izz="0.0013315199498696443" ixy="0.0" iyz="0.0" ixz="0.0" />
     </inertial>
     <visual>
-      <origin xyz="0 0 0" rpy="0 0 0" />
+      <origin xyz="0 0 0" rpy="0 0 ${pi/2}" />
       <geometry>
         <mesh filename="package://waver_description/meshes/base_link.stl" scale="${scale}" />
@@ -22,5 +22,5 @@
     </visual>
     <collision>
-      <origin xyz="0 0 0" rpy="0 0 0" />
+      <origin xyz="0 0 0" rpy="0 0 ${pi/2}" />
       <geometry>
         <mesh filename="package://waver_description/meshes/base_link.stl" scale="${scale}" />
@@ -31,9 +31,9 @@
     <inertial>
       <mass value="${mass_top}" />
-      <origin xyz="${mass_center_top}" rpy="0 0 0" />
+      <origin xyz="${mass_center_top}" rpy="0 0 ${pi/2}" />
       <inertia ixx="0.0022122780308922725" iyy="0.0018048674350663336" izz="0.003659349844340526" ixy="0.0" iyz="0.0" ixz="0.0" />
     </inertial>
     <visual>
-      <origin xyz="0 0 0" rpy="0 0 0" />
+      <origin xyz="0 0 0" rpy="0 0 ${pi/2}" />
       <geometry>
         <mesh filename="package://waver_description/meshes/top_shell_link.stl" scale="${scale}" />
@@ -42,5 +42,5 @@
     </visual>
     <collision>
-      <origin xyz="0 0 0" rpy="0 0 0" />
+      <origin xyz="0 0 0" rpy="0 0 ${pi/2}" />
       <geometry>
         <mesh filename="package://waver_description/meshes/top_shell_link.stl" scale="${scale}" />
@@ -51,9 +51,9 @@
     <inertial>
       <mass value="${mass_acces}" />
-      <origin xyz="${mass_center_acces}" rpy="0 0 0" />
+      <origin xyz="${mass_center_acces}" rpy="0 0 ${pi/2}" />
       <inertia ixx="2.2622278969724113e-07" iyy="7.36227380617578e-07" izz="7.362274117066844e-07" ixy="0.0" iyz="0.0" ixz="0.0" />
     </inertial>
     <visual>
-      <origin xyz="${position_acces}" rpy="0 0 0" />
+      <origin xyz="${position_acces}" rpy="0 0 ${pi/2}" />
       <geometry>
         <mesh filename="package://waver_description/meshes/accessories_link.stl" scale="${scale}" />
@@ -62,5 +62,5 @@
     </visual>
     <collision>
-      <origin xyz="${position_acces}" rpy="0 0 0" />
+      <origin xyz="${position_acces}" rpy="0 0 ${pi/2}" />
       <geometry>
         <mesh filename="package://waver_description/meshes/accessories_link.stl" scale="${scale}" />
@@ -71,9 +71,9 @@
     <inertial>
       <mass value="${mass_acces1}" />
-      <origin xyz="${mass_center_acces1}" rpy="0 0 0" />
+      <origin xyz="${mass_center_acces1}" rpy="0 0 ${pi/2}" />
       <inertia ixx="1.8160055789601745e-07" iyy="8.100907081280738e-07" izz="8.100806017664777e-07" ixy="0.0" iyz="0.0" ixz="0.0" />
     </inertial>
     <visual>
-      <origin xyz="${position_acces1}" rpy="0 0 0" />
+      <origin xyz="${position_acces1}" rpy="0 0 ${pi/2}" />
       <geometry>
         <mesh filename="package://waver_description/meshes/accessories1_link.stl" scale="${scale}" />
@@ -82,5 +82,5 @@
     </visual>
     <collision>
-      <origin xyz="${position_acces1}" rpy="0 0 0" />
+      <origin xyz="${position_acces1}" rpy="0 0 ${pi/2}" />
       <geometry>
         <mesh filename="package://waver_description/meshes/accessories1_link.stl" scale="${scale}" />
@@ -91,9 +91,9 @@
     <inertial>
       <mass value="${mass_board}" />
-      <origin xyz="${mass_center_board}" rpy="0 0 0" />
+      <origin xyz="${mass_center_board}" rpy="0 0 ${pi/2}" />
       <inertia ixx="5.313564367625195e-06" iyy="5.192849578266062e-06" izz="8.832425081682543e-06" ixy="0.0" iyz="0.0" ixz="0.0" />
     </inertial>
     <visual>
-      <origin xyz="${position_board}" rpy="0 0 0" />
+      <origin xyz="${position_board}" rpy="0 0 ${pi/2}" />
       <geometry>
         <mesh filename="package://waver_description/meshes/board_link.stl" scale="${scale}" />
@@ -102,5 +102,5 @@
     </visual>
     <collision>
-      <origin xyz="${position_board}" rpy="0 0 0" />
+      <origin xyz="${position_board}" rpy="0 0 ${pi/2}" />
       <geometry>
         <mesh filename="package://waver_description/meshes/board_link.stl" scale="${scale}" />
@@ -111,9 +111,9 @@
     <inertial>
       <mass value="${mass_screen}" />
-      <origin xyz="${mass_center_screen}" rpy="0 0 0" />
+      <origin xyz="${mass_center_screen}" rpy="0 0 ${pi/2}" />
       <inertia ixx="3.186534864702538e-08" iyy="2.5666330224105178e-07" izz="2.7215400443770056e-07" ixy="0.0" iyz="0.0" ixz="0.0" />
     </inertial>
     <visual>
-      <origin xyz="${position_screen}" rpy="0 0 0" />
+      <origin xyz="${position_screen}" rpy="0 0 ${pi/2}" />
       <geometry>
         <mesh filename="package://waver_description/meshes/oled_screen_link.stl" scale="${scale}" />
@@ -122,5 +122,5 @@
     </visual>
     <collision>
-      <origin xyz="${position_screen}" rpy="0 0 0" />
+      <origin xyz="${position_screen}" rpy="0 0 ${pi/2}" />
       <geometry>
         <mesh filename="package://waver_description/meshes/oled_screen_link.stl" scale="${scale}" />
@@ -131,9 +131,9 @@
     <inertial>
       <mass value="${mass_wbl}" />
-      <origin xyz="0 0 0" rpy="0 0 0" />
+      <origin xyz="0 0 0" rpy="0 0 ${pi/2}" />
       <inertia ixx="0.0011153598236428852" iyy="0.0007115715200341761" izz="0.0007099489264864056" ixy="0.0" iyz="0.0" ixz="0.0" />
     </inertial>
     <visual>
-      <origin xyz="${position_wbl}" rpy="0 0 0" />
+      <origin xyz="${position_wbl}" rpy="0 0 ${pi/2}" />
       <geometry>
         <mesh filename="package://waver_description/meshes/wheel_back_left_link.stl" scale="${scale}" />
@@ -142,5 +142,5 @@
     </visual>
     <collision>
-      <origin xyz="${position_wbl}" rpy="0 0 0" />
+      <origin xyz="${position_wbl}" rpy="0 0 ${pi/2}" />
       <geometry>
         <mesh filename="package://waver_description/meshes/wheel_back_left_link.stl" scale="${scale}" />
@@ -151,9 +151,9 @@
     <inertial>
       <mass value="${mass_wfl}" />
-      <origin xyz="0 0 0" rpy="0 0 0" />
+      <origin xyz="0 0 0" rpy="0 0 ${pi/2}" />
       <inertia ixx="0.0011153873944048257" iyy="0.0007115715200341761" izz="0.0007099764972483459" ixy="0.0" iyz="0.0" ixz="0.0" />
     </inertial>
     <visual>
-      <origin xyz="${position_wfl}" rpy="0 0 0" />
+      <origin xyz="${position_wfl}" rpy="0 0 ${pi/2}" />
       <geometry>
         <mesh filename="package://waver_description/meshes/wheel_front_left_link.stl" scale="${scale}" />
@@ -162,5 +162,5 @@
     </visual>
     <collision>
-      <origin xyz="${position_wfl}" rpy="0 0 0" />
+      <origin xyz="${position_wfl}" rpy="0 0 ${pi/2}" />
       <geometry>
         <mesh filename="package://waver_description/meshes/wheel_front_left_link.stl" scale="${scale}" />
@@ -171,9 +171,9 @@
     <inertial>
       <mass value="${mass_wfr}" />
-      <origin xyz="0 0 0" rpy="0 0 0" />
+      <origin xyz="0 0 0" rpy="0 0 ${pi/2}" />
       <inertia ixx="0.0011153598236428852" iyy="0.0007115715475157099" izz="0.0007099489539679392" ixy="0.0" iyz="0.0" ixz="0.0" />
     </inertial>
     <visual>
-      <origin xyz="${position_wfr}" rpy="0 0 0" />
+      <origin xyz="${position_wfr}" rpy="0 0 ${pi/2}" />
       <geometry>
         <mesh filename="package://waver_description/meshes/wheel_front_right_link.stl" scale="${scale}" />
@@ -182,5 +182,5 @@
     </visual>
     <collision>
-      <origin xyz="${position_wfr}" rpy="0 0 0" />
+      <origin xyz="${position_wfr}" rpy="0 0 ${pi/2}" />
       <geometry>
         <mesh filename="package://waver_description/meshes/wheel_front_right_link.stl" scale="${scale}" />
@@ -191,9 +191,9 @@
     <inertial>
       <mass value="${mass_wbr}" />
-      <origin xyz="0 0 0" rpy="0 0 0" />
+      <origin xyz="0 0 0" rpy="0 0 ${pi/2}" />
       <inertia ixx="0.0011153873944048257" iyy="0.0007115715475157099" izz="0.0007099765247298796" ixy="0.0" iyz="0.0" ixz="0.0" />
     </inertial>
     <visual>
-      <origin xyz="${position_wbr}" rpy="0 0 0" />
+      <origin xyz="${position_wbr}" rpy="0 0 ${pi/2}" />
       <geometry>
         <mesh filename="package://waver_description/meshes/wheel_back_right_link.stl" scale="${scale}" />
@@ -202,5 +202,5 @@
     </visual>
     <collision>
-      <origin xyz="${position_wbr}" rpy="0 0 0" />
+      <origin xyz="${position_wbr}" rpy="0 0 ${pi/2}" />
       <geometry>
         <mesh filename="package://waver_description/meshes/wheel_back_right_link.stl" scale="${scale}" />
@@ -221,70 +221,46 @@
   </joint>
   <joint name="top_acces_joint" type="fixed">
-    <origin xyz="${mass_center_acces}" rpy="0 0 0" />
+    <origin xyz="${positions_acces_joint}" rpy="0 0 0" />
     <parent link="top_shell_link" />
     <child link="accessories_link" />
   </joint>
-  <joint name="top_acces1_joint" type="fixed">
-    <origin xyz="${mass_center_acces1}" rpy="0 0 0" />
+<joint name="top_acces1_joint" type="fixed">
+    <origin xyz="${positions_acces1_joint}" rpy="0 0 0" />
     <parent link="top_shell_link" />
     <child link="accessories1_link" />
   </joint>
   <joint name="top_board_joint" type="fixed">
-    <origin xyz="${mass_center_board}" rpy="0 0 0" />
+    <origin xyz="${positions_board_joint}" rpy="0 0 0" />
     <parent link="top_shell_link" />
     <child link="board_link" />
   </joint>
   <joint name="top_screen_joint" type="fixed">
-    <origin xyz="${mass_center_screen}" rpy="0 0 0" />
+    <origin xyz="${positions_screen_joint}" rpy="0 0 0" />
     <parent link="top_shell_link" />
     <child link="oled_screen_link" />
   </joint>
   <joint name="wheel_back_left_joint" type="continuous">
-    <origin xyz="${mass_center_wbl}" rpy="0 0 0" />
+    <origin xyz="${position_wbl_joint}" rpy="0 0 0" />
     <parent link="base_link" />
     <child link="wheel_back_left_link" />
-    <axis xyz="1 0 0" />
+    <axis xyz="0 1 0" />
   </joint>
   <joint name="wheel_front_left_joint" type="continuous">
-    <origin xyz="${mass_center_wfl}" rpy="0 0 0" />
+    <origin xyz="${position_wfl_joint}" rpy="0 0 0" />
     <parent link="base_link" />
     <child link="wheel_front_left_link" />
-    <axis xyz="1 0 0" />
+    <axis xyz="0 1 0" />
   </joint>
   <joint name="wheel_front_right_joint" type="continuous">
-    <origin xyz="${mass_center_wfr}" rpy="0 0 0" />
+    <origin xyz="${position_wfr_joint}" rpy="0 0 0" />
     <parent link="base_link" />
     <child link="wheel_front_right_link" />
-    <axis xyz="1 0 0" />
+    <axis xyz="0 1 0" />
   </joint>
   <joint name="wheel_back_right_joint" type="continuous">
-    <origin xyz="${mass_center_wbr}" rpy="0 0 0" />
+    <origin xyz="${position_wbr_joint}" rpy="0 0 0" />
     <parent link="base_link" />
     <child link="wheel_back_right_link" />
-    <axis xyz="1 0 0" />
-  </joint>
-  <gazebo>
-    <plugin name="skid_steer_drive_controller" filename="libgazebo_ros_skid_steer_drive.so">
-      <robotNamespace></robotNamespace>
-      <updateRate>100.0</updateRate>
-      <leftFrontJoint>wheel_front_left_joint</leftFrontJoint>
-      <rightFrontJoint>wheel_front_right_joint</rightFrontJoint>
-      <leftRearJoint>wheel_back_left_joint</leftRearJoint>
-      <rightRearJoint>wheel_back_right_joint</rightRearJoint>
-      <wheelSeparation>${wheel_separation}</wheelSeparation>
-      <wheelDiameter>${2*wheel_radius}</wheelDiameter>
-      <torque>2</torque>
-      <commandTopic>cmd_vel</commandTopic>
-      <odometryTopic>odom</odometryTopic>
-      <odometryFrame>odom</odometryFrame>
-      <robotBaseFrame>base_footprint</robotBaseFrame>
-      <publishWheelTF>true</publishWheelTF>
-      <publishOdom>true</publishOdom>
-      <publishWheelJointState>true</publishWheelJointState>
-      <covariance_x>0.0001</covariance_x>
-      <covariance_y>0.0001</covariance_y>
-      <covariance_yaw>0.01</covariance_yaw>
-      <broadcastTF>true</broadcastTF>
-    </plugin>
-  </gazebo>
+    <axis xyz="0 1 0" />
+  </joint>
 </robot>
